Commit message: Another commit

File: franka_description/robots/panda_arm.urdf.xacro (robot description, xacro)
@@ -5,12 +5,19 @@
   <xacro:arg name="robot_ip" default=""/> <!-- IP address or hostname of the robot" -->
   <xacro:arg name="use_fake_hardware" default="false"/>
+  <xacro:arg name="use_sim" default="true"/>
   <xacro:arg name="fake_sensor_commands" default="false"/>
-  <xacro:include filename="$(find franka_description)/robots/panda_arm.xacro"/>
-  <xacro:panda_arm arm_id="$(arg arm_id)" safety_distance="0.03"/>
-  <xacro:if value="$(arg hand)">
-    <xacro:include filename="$(find franka_description)/robots/hand.xacro"/>
+  <xacro:include filename="$(find franka_description)/urdf/panda_arm.xacro"/>
+  <xacro:panda_arm arm_id="$(arg arm_id)" safety_distance="0.001"/>
+  <!-- <xacro:if value="$(arg hand)">
+    <xacro:include filename="$(find franka_description)/urdf/hand.xacro"/>
     <xacro:hand ns="$(arg arm_id)" rpy="0 0 ${-pi/4}" connected_to="$(arg arm_id)_link8" safety_distance="0.03"/>
+  </xacro:if> -->
+  <!-- <xacro:include filename="$(find franka_description)/urdf/panda_arm.ros2_control.xacro"/>
+  <xacro:panda_arm_ros2_control arm_id="$(arg arm_id)" robot_ip="$(arg robot_ip)" use_fake_hardware="$(arg use_fake_hardware)" use_sim="$(arg use_sim)" fake_sensor_commands="$(arg fake_sensor_commands)"/> -->
+  <xacro:include filename="$(find franka_description)/urdf/panda_arm.ros2_control2.xacro"/>
+  <xacro:panda_ros2control prefix="$(arg arm_id)" EE_no="true"/>
+  <xacro:if value="$(arg use_sim)">
+    <xacro:include filename="$(find franka_description)/urdf/panda_arm.transmission.xacro"/>
+    <xacro:panda_transmission arm_id="$(arg arm_id)"/>
   </xacro:if>
-  <xacro:include filename="$(find franka_description)/robots/panda_arm.ros2_control.xacro"/>
-  <xacro:panda_arm_ros2_control ns="$(arg arm_id)" robot_ip="$(arg robot_ip)" use_fake_hardware="$(arg use_fake_hardware)" fake_sensor_commands="$(arg fake_sensor_commands)"/>
 </robot>

File: franka_description/urdf/panda_arm.xacro (robot description, xacro)
@@ -3,6 +3,7 @@
   <!-- safety_distance: Minimum safety distance in [m] by which the collision volumes are expanded and which is enforced during robot motions -->
   <!-- arm_id: Namespace of the panda arm. Serves to differentiate between arms in case of multiple instances. -->
-  <xacro:macro name="panda_arm" params="arm_id:='panda' description_pkg:='franka_description' connected_to:='' xyz:='0 0 0' rpy:='0 0 0' safety_distance:=0">
+  <xacro:macro name="panda_arm" params="arm_id:='panda' description_pkg:='franka_description' connected_to:='world' xyz:='0 0 0' rpy:='0 0 0' safety_distance:=0">
     <xacro:unless value="${not connected_to}">
+      <link name="${connected_to}"/>
       <joint name="${arm_id}_joint_${connected_to}" type="fixed">
         <parent link="${connected_to}"/>
@@ -12,10 +13,18 @@
     </xacro:unless>
     <link name="${arm_id}_link0">
-      <visual>
-        <geometry>
-          <mesh filename="package://${description_pkg}/meshes/visual/link0.dae"/>
-        </geometry>
-      </visual>
-      <collision>
+      <inertial>
+        <mass value="2.92"/>
+        <origin rpy="0 0 0" xyz="-0.025566 -2.88e-05 0.057332"/>
+        <inertia ixx="0.00782229414331" ixy="-1.56191622996e-05" ixz="-0.00126005738123" iyy="0.0109027971813" iyz="1.08233858202e-05" izz="0.0102355503949"/>
+      </inertial>
+      <visual>
+        <geometry>
+          <mesh filename="file://$(find ${description_pkg})/meshes/visual/link0.dae"/>
+        </geometry>
+        <material name="">
+          <color rgba="1 1 1 1"/>
+        </material>
+      </visual>
+      <!-- <collision>
         <origin xyz="-0.075 0 0.06" rpy="0 ${pi/2} 0"/>
         <geometry>
@@ -34,28 +43,45 @@
           <sphere radius="${0.06+safety_distance}" />
         </geometry>
+      </collision>  -->
+      <collision>
+        <origin rpy="0 0 0" xyz="0 0 0"/>
+        <geometry>
+          <mesh filename="file://$(find ${description_pkg})/meshes/collision/link0.stl"/>
+        </geometry>
       </collision>
     </link>
     <link name="${arm_id}_link1">
-      <visual>
-        <geometry>
-          <mesh filename="package://${description_pkg}/meshes/visual/link1.dae"/>
-        </geometry>
-      </visual>
-      <collision>
+      <inertial>
+        <mass value="2.74"/>
+        <origin rpy="0 0 0" xyz="0 -0.0324958 -0.0675818"/>
+        <inertia ixx="0.0180416958283" ixy="0.0" ixz="0.0" iyy="0.0159136071891" iyz="0.0046758424612" izz="0.00620690827127"/>
+      </inertial>
+      <visual>
+        <geometry>
+          <mesh filename="file://$(find ${description_pkg})/meshes/visual/link1.dae"/>
+        </geometry>
+      </visual>
+      <!-- <collision>
         <origin xyz="0 0 -0.1915" rpy="0 0 0"/>
         <geometry>
-          <cylinder radius="${0.06+safety_distance}" length="0.2830" />
-        </geometry>
-      </collision>
-      <collision>
+          <cylinder radius="${0.06+safety_distance}" length="0.1830" />
+        </geometry>
+      </collision>
+      <collision>
+        <origin xyz="0 0 -0.05" rpy="0 0 0"/>
+        <geometry>
+          <sphere radius="${0.06+safety_distance}" />
+        </geometry>
+      </collision> -->
+      <!-- <collision>
         <origin xyz="0 0 -0.333" rpy="0 0 0"/>
         <geometry>
           <sphere radius="${0.06+safety_distance}" />
         </geometry>
-      </collision>
-      <collision>
-        <origin xyz="0 0 -0.05" rpy="0 0 0"/>
-        <geometry>
-          <sphere radius="${0.06+safety_distance}" />
+      </collision> -->
+      <collision>
+        <origin rpy="0 0 0" xyz="0 0 0"/>
+        <geometry>
+          <mesh filename="file://$(find ${description_pkg})/meshes/collision/link1.stl"/>
         </geometry>
       </collision>
@@ -68,12 +94,18 @@
       <axis xyz="0 0 1"/>
       <limit effort="87" lower="-2.8973" upper="2.8973" velocity="2.1750"/>
+      <!-- <dynamics damping="50.0" friction="1.0"/> -->
     </joint>
     <link name="${arm_id}_link2">
-      <visual>
-        <geometry>
-          <mesh filename="package://${description_pkg}/meshes/visual/link2.dae"/>
-        </geometry>
-      </visual>
-      <collision>
+      <inertial>
+        <mass value="2.74"/>
+        <origin rpy="0 0 0" xyz="0 -0.06861 0.0322285"/>
+        <inertia ixx="0.0182856182281" ixy="0.0" ixz="0.0" iyy="0.00621358421175" iyz="-0.00472844221905" izz="0.0161514346309"/>
+      </inertial>
+      <visual>
+        <geometry>
+          <mesh filename="file://$(find ${description_pkg})/meshes/visual/link2.dae"/>
+        </geometry>
+      </visual>
+      <!-- <collision>
         <origin xyz="0 0 0" rpy="0 0 0"/>
         <geometry>
@@ -91,4 +123,10 @@
         <geometry>
           <sphere radius="${0.06+safety_distance}" />
+        </geometry>
+      </collision> -->
+      <collision>
+        <origin rpy="0 0 0" xyz="0 0 0"/>
+        <geometry>
+          <mesh filename="file://$(find ${description_pkg})/meshes/collision/link2.stl"/>
         </geometry>
       </collision>
@@ -101,12 +139,18 @@
       <axis xyz="0 0 1"/>
       <limit effort="87" lower="-1.7628" upper="1.7628" velocity="2.1750"/>
+      <dynamics damping="50.0" friction="1.0"/>
     </joint>
     <link name="${arm_id}_link3">
-      <visual>
-        <geometry>
-          <mesh filename="package://${description_pkg}/meshes/visual/link3.dae"/>
-        </geometry>
-      </visual>
-      <collision>
+      <inertial>
+        <mass value="2.38"/>
+        <origin rpy="0 0 0" xyz="0.0469893 0.0316374 -0.031704"/>
+        <inertia ixx="0.00771376630908" ixy="-0.00248490625138" ixz="-0.00332147581033" iyy="0.00989108008727" iyz="-0.00217796151484" izz="0.00811723558464"/>
+      </inertial>
+      <visual>
+        <geometry>
+          <mesh filename="file://$(find ${description_pkg})/meshes/visual/link3.dae"/>
+        </geometry>
+      </visual>
+      <!-- <collision>
         <origin xyz="0 0 -0.145" rpy="0 0 0"/>
         <geometry>
@@ -124,4 +168,10 @@
         <geometry>
           <sphere radius="${0.06+safety_distance}" />
+        </geometry>
+      </collision> -->
+      <collision>
+        <origin rpy="0 0 0" xyz="0 0 0"/>
+        <geometry>
+          <mesh filename="file://$(find ${description_pkg})/meshes/collision/link3.stl"/>
         </geometry>
       </collision>
@@ -134,12 +184,18 @@
       <axis xyz="0 0 1"/>
       <limit effort="87" lower="-2.8973" upper="2.8973" velocity="2.1750"/>
+      <dynamics damping="10.0" friction="1.0"/>
     </joint>
     <link name="${arm_id}_link4">
-      <visual>
-        <geometry>
-          <mesh filename="package://${description_pkg}/meshes/visual/link4.dae"/>
-        </geometry>
-      </visual>
-      <collision>
+      <inertial>
+        <mass value="2.38"/>
+        <origin rpy="0 0 0" xyz="-0.0360446 0.0336853 0.031882"/>
+        <inertia ixx="0.00799663881132" ixy="0.00347095570217" ixz="-0.00241222942995" iyy="0.00825390705278" iyz="0.00235774044121" izz="0.0102515004345"/>
+      </inertial>
+      <visual>
+        <geometry>
+          <mesh filename="file://$(find ${description_pkg})/meshes/visual/link4.dae"/>
+        </geometry>
+      </visual>
+      <!-- <collision>
         <origin xyz="0 0 0" rpy="0 0 0"/>
         <geometry>
@@ -157,4 +213,10 @@
         <geometry>
           <sphere radius="${0.06+safety_distance}" />
+        </geometry>
+      </collision> -->
+      <collision>
+        <origin rpy="0 0 0" xyz="0 0 0"/>
+        <geometry>
+          <mesh filename="file://$(find ${description_pkg})/meshes/collision/link4.stl"/>
         </geometry>
       </collision>
@@ -166,13 +228,20 @@
       <child link="${arm_id}_link4"/>
       <axis xyz="0 0 1"/>
-      <limit effort="87" lower="-3.0718" upper="-0.0698" velocity="2.1750"/>
+      <limit effort="87" lower="-3.0718" upper="0.0698" velocity="2.1750"/>
+      <!-- upper should be -0.0698, but that brakes simulation when initial position for this joint is 0.0 -->
+      <dynamics damping="10.0" friction="1.0"/>
     </joint>
     <link name="${arm_id}_link5">
-      <visual>
-        <geometry>
-          <mesh filename="package://${description_pkg}/meshes/visual/link5.dae"/>
-        </geometry>
-      </visual>
-      <collision>
+      <inertial>
+        <mass value="2.74"/>
+        <origin rpy="0 0 0" xyz="0 0.0610427 -0.104176"/>
+        <inertia ixx="0.030371374513" ixy="6.50283587108e-07" ixz="-1.05129179916e-05" iyy="0.0288752887402" iyz="-0.00775653445787" izz="0.00444134056164"/>
+      </inertial>
+      <visual>
+        <geometry>
+          <mesh filename="file://$(find ${description_pkg})/meshes/visual/link5.dae"/>
+        </geometry>
+      </visual>
+      <!-- <collision>
         <origin xyz="0 0 -0.26" rpy="0 0 0"/>
         <geometry>
@@ -208,4 +277,10 @@
         <geometry>
           <sphere radius="${0.025+safety_distance}" />
+        </geometry>
+      </collision> -->
+      <collision>
+        <origin rpy="0 0 0" xyz="0 0 0"/>
+        <geometry>
+          <mesh filename="file://$(find ${description_pkg})/meshes/collision/link5.stl"/>
         </geometry>
       </collision>
@@ -218,12 +293,18 @@
       <axis xyz="0 0 1"/>
       <limit effort="12" lower="-2.8973" upper="2.8973" velocity="2.6100"/>
+      <dynamics damping="5.0" friction="1.0"/>
     </joint>
     <link name="${arm_id}_link6">
-      <visual>
-        <geometry>
-          <mesh filename="package://${description_pkg}/meshes/visual/link6.dae"/>
-        </geometry>
-      </visual>
-      <collision>
+      <inertial>
+        <mass value="1.55"/>
+        <origin rpy="0 0 0" xyz="0.0510509 0.009108 0.0106343"/>
+        <inertia ixx="0.00303336450376" ixy="-0.000437276865508" ixz="0.000629257294877" iyy="0.00404479911567" iyz="0.000130472021025" izz="0.00558234286039"/>
+      </inertial>
+      <visual>
+        <geometry>
+          <mesh filename="file://$(find ${description_pkg})/meshes/visual/link6.dae"/>
+        </geometry>
+      </visual>
+      <!-- <collision>
         <origin xyz="0 0 -0.03" rpy="0 0 0"/>
         <geometry>
@@ -241,4 +322,10 @@
         <geometry>
           <sphere radius="${0.05+safety_distance}" />
+        </geometry>
+      </collision> -->
+      <collision>
+        <origin rpy="0 0 0" xyz="0 0 0"/>
+        <geometry>
+          <mesh filename="file://$(find ${description_pkg})/meshes/collision/link6.stl"/>
         </geometry>
       </collision>
@@ -251,12 +338,18 @@
       <axis xyz="0 0 1"/>
       <limit effort="12" lower="-0.0175" upper="3.7525" velocity="2.6100"/>
+      <dynamics damping="5.0" friction="1.0"/>
     </joint>
     <link name="${arm_id}_link7">
-      <visual>
-        <geometry>
-          <mesh filename="package://${description_pkg}/meshes/visual/link7.dae"/>
-        </geometry>
-      </visual>
-      <collision>
+      <inertial>
+        <mass value="0.54"/>
+        <origin rpy="0 0 0" xyz="0.0109695 0.0107965 0.0650411"/>
+        <inertia ixx="0.000888868887021" ixy="-0.00012239074652" ixz="3.98699829666e-05" iyy="0.000888001373233" iyz="-9.33825115206e-05" izz="0.0007176834609"/>
+      </inertial>
+      <visual>
+        <geometry>
+          <mesh filename="file://$(find ${description_pkg})/meshes/visual/link7.dae"/>
+        </geometry>
+      </visual>
+      <!-- <collision>
         <origin xyz="0 0 0.01" rpy="0 0 0"/>
         <geometry>
@@ -274,4 +367,10 @@
         <geometry>
           <sphere radius="${0.04+safety_distance}"  />
+        </geometry>
+      </collision> -->
+      <collision>
+        <origin rpy="0 0 0" xyz="0 0 0"/>
+        <geometry>
+          <mesh filename="file://$(find ${description_pkg})/meshes/collision/link7.stl"/>
         </geometry>
       </collision>
@@ -284,7 +383,8 @@
       <axis xyz="0 0 1"/>
       <limit effort="12" lower="-2.8973" upper="2.8973" velocity="2.6100"/>
+      <dynamics damping="1.0" friction="1.0"/>
     </joint>
     <link name="${arm_id}_link8">
-      <collision>
+      <!-- <collision>
         <origin xyz="0.0424 0.0424 -0.0250" rpy="${pi} ${pi/2} ${pi/2}"/>
         <geometry>
@@ -303,5 +403,5 @@
           <sphere radius="${0.03+safety_distance}"  />
         </geometry>
-      </collision>
+      </collision> -->
     </link>
     <joint name="${arm_id}_joint8" type="fixed">
